Commit message: fixed Linux build; fixed simulation run on slower machines/vms; an attempt to make motion control work

File: platform/src/openvmp_robot_don1/models/openvmp_robot_don1.urdf (robot description, URDF)
Before this commit: robot openvmp_robot_don1, 2 links, 1 joints
Links:
- added link base_link2; collision box size=${base_length/2} ${base_width} ${base_height/2}; visual box size=${base_length/2} ${base_width} ${base_height/2}
- link base_link: geometry collision box size=${base_length} ${base_width} ${base_height/2}; visual box size=${base_length} ${base_width} ${base_height/2}
Joints:
- added joint base_joint2: type fixed, parent base_link, child base_link2, origin xyz=0.0 0.0 ${base_height/2} rpy=0 0 0
- joint base_joint: origin xyz=0.0 0.0 0.0 rpy=0 0 0 -> xyz=0.0 0.0 1.0 rpy=0 0 0

Commit message: Use rendered meshes in the simulation.

File: platform/src/openvmp_robot_don1/models/openvmp_robot_don1.urdf (robot description, URDF)
Before this commit: robot openvmp_robot_don1, 3 links, 2 joints
Links:
- removed link base_link2
- link base_link: geometry collision box size=${base_length/2} ${base_width} ${base_height/2}; collision box size=${base_length} ${base_width} ${base_height/2}
Joints:
- removed joint base_joint2
- joint base_joint: origin xyz=0.0 0.0 1.0 rpy=0 0 0 -> xyz=0.0 0.0 0.0 rpy=0 0 0
